File: hotfire_pcbs/TC-board/TC-board.kicad_sch (KiCad schematic)
At the start: 13 parts, among them J1 DB15_Female, J3 PCIE-LP-01-01-F-DV-A-TR, U1 MAX31856_Breakout, U2 MAX31856_Breakout

Commit message: Fixed card edge clearance violation
Parts:
- J3: footprint Connector_PCBEdge:BUS_PCIexpress_x1 -> PCIe_x1_card_edge:PCIe_x1_card_edge
Changed lines of the file:
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@@
       (effects (font (size 1.27 1.27)) (justify left bottom))
     )
-    (property "Footprint" "Connector_PCBEdge:BUS_PCIexpress_x1" (id 2) (at 100.584 116.84 0)
+    (property "Footprint" "PCIe_x1_card_edge:PCIe_x1_card_edge" (id 2) (at 100.584 116.84 0)
       (effects (font (size 1.27 1.27)) hide)
     )
@@
     )
     (path "/19e0a432-371a-451a-988e-c01fc4d96ec9"
-      (reference "J3") (unit 1) (value "PCIE-LP-01-01-F-DV-A-TR") (footprint "Connector_PCBEdge:BUS_PCIexpress_x1")
+      (reference "J3") (unit 1) (value "PCIE-LP-01-01-F-DV-A-TR") (footprint "PCIe_x1_card_edge:PCIe_x1_card_edge")
     )
     (path "/247c8275-c689-4ade-a534-8ec2fd4f463e"
